File: FT232.brd (EAGLE design)
At the start: 100 x 80 mm, 17 parts, among them J1 USB, J2 CON, U1 FT232, Y1 CRYSTAL

Commit message: 第一次布线尝试
Parts:
- moved Z1 5.08 mm to (17.8, 5.08)
- moved R3 2.54 mm to (14.0, 7.62)
- moved Z2 2.54 mm to (17.8, 7.62)
- moved Z3 2.54 mm to (17.8, 10.2)
- moved C4 2.54 mm to (14.0, 6.35)
- moved R4 1.27 mm to (14.0, 8.89)
- moved R1 1.27 mm to (14.0, 3.81)
- moved R2 1.27 mm to (14.0, 5.08)
- moved R5 1.27 mm to (14.0, 10.2)
Routing:
- net +5V: track 0.00 -> 64.4 mm, vias 0 -> 2
- net RXD: track 0.00 -> 13.8 mm, vias 0 -> 1
- net N$8: track 0.00 -> 12.8 mm, vias 0 -> 2
- net N$9: track 0.00 -> 10.6 mm, vias 0 -> 2
- net TXD: track 0.00 -> 10.2 mm, vias 0 -> 1
- net N$3: track 0.00 -> 9.94 mm
- net N$7: track 0.00 -> 9.89 mm
- net N$4: track 0.00 -> 9.87 mm
- net N$1: track 0.00 -> 9.57 mm
- net N$6: track 0.00 -> 9.32 mm
- net N$2: track 0.00 -> 8.72 mm
- net N$5: track 0.00 -> 8.45 mm
- net GND: track 0.00 -> 6.05 mm, vias 0 -> 8
- net N$12: track 0.00 -> 4.60 mm, vias 0 -> 2
- net N$11: track 0.00 -> 2.74 mm
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- added copper zone on layer 1, net GND
- added copper zone on layer 16, net GND

Commit message: 边界
Other:
- board size 100 x 80 mm -> 37.5 x 12 mm
Changed lines of the file:
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@@
 <board>
 <plain>
-<wire x1="0" y1="0" x2="100" y2="0" width="0" layer="20"/>
-<wire x1="100" y1="0" x2="100" y2="80" width="0" layer="20"/>
-<wire x1="100" y1="80" x2="0" y2="80" width="0" layer="20"/>
-<wire x1="0" y1="80" x2="0" y2="0" width="0" layer="20"/>
 <wire x1="2.1082" y1="13.6144" x2="39.624" y2="13.6144" width="0.127" layer="20"/>
 <wire x1="39.624" y1="13.6144" x2="39.624" y2="1.6256" width="0.127" layer="21"/>
