File: FT232.sch (EAGLE design)
At the start: 17 parts, among them J1 USB, J2 CON, U1 FT232, Y1 CRYSTAL

Commit message: 第二次布线尝试
Parts:
- J1: value USB -> USBA; device FT232:USB -> FT232:USBA
Connections:
- net N$1 renamed D_N
- net N$2 renamed D_P
Other:
- moved on the sheet: J1
Changed lines of the file:
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@@
 <parts>
 <part name="U1" library="FT232" deviceset="FT232" device=""/>
-<part name="J1" library="FT232" deviceset="USB" device=""/>
 <part name="J2" library="FT232" deviceset="CON" device=""/>
 <part name="Y1" library="FT232" deviceset="CRYSTAL" device=""/>
@@
 <part name="GND7" library="supply1" deviceset="GND" device=""/>
 <part name="GND8" library="supply1" deviceset="GND" device=""/>
+<part name="J1" library="FT232" deviceset="USB" device="A"/>
 </parts>
 <sheets>
@@
 <instances>
 <instance part="U1" gate="A" x="137.16" y="101.6"/>
-<instance part="J1" gate="A" x="48.26" y="111.76"/>
 <instance part="J2" gate="A" x="236.22" y="111.76"/>
 <instance part="Y1" gate="A" x="93.98" y="93.98"/>
@@
 <instance part="GND7" gate="1" x="205.74" y="88.9"/>
 <instance part="GND8" gate="1" x="99.06" y="121.92" rot="R270"/>
+<instance part="J1" gate="A" x="48.26" y="111.76"/>
 </instances>
 <busses>
 </busses>
 <nets>
-<net name="N$1" class="0">
+<net name="D_N" class="0">
 <segment>
 <pinref part="R1" gate="A" pin="2"/>
@@
 </segment>
 </net>
-<net name="N$2" class="0">
+<net name="D_P" class="0">
 <segment>
 <pinref part="U1" gate="A" pin="USBDP"/>
@@
 <segment>
 <pinref part="R1" gate="A" pin="1"/>
+<wire x1="86.36" y1="114.3" x2="60.96" y2="114.3" width="0.1524" layer="91"/>
 <pinref part="J1" gate="A" pin="D-"/>
-<wire x1="86.36" y1="114.3" x2="60.96" y2="114.3" width="0.1524" layer="91"/>
 </segment>
 </net>
 <net name="N$4" class="0">
 <segment>
-<pinref part="J1" gate="A" pin="D+"/>
 <pinref part="R2" gate="A" pin="1"/>
 <wire x1="60.96" y1="111.76" x2="86.36" y2="111.76" width="0.1524" layer="91"/>
+<pinref part="J1" gate="A" pin="D+"/>
 </segment>
 </net>
@@
 <net name="GND" class="0">
 <segment>
-<pinref part="J1" gate="A" pin="GND"/>
 <pinref part="GND1" gate="1" pin="GND"/>
 <wire x1="60.96" y1="106.68" x2="66.04" y2="106.68" width="0.1524" layer="91"/>
 <wire x1="66.04" y1="106.68" x2="66.04" y2="101.6" width="0.1524" layer="91"/>
+<pinref part="J1" gate="A" pin="GND"/>
 </segment>
 <segment>
@@
 <net name="+5V" class="0">
 <segment>
-<pinref part="J1" gate="A" pin="VBUS"/>
+<pinref part="R5" gate="A" pin="2"/>
+<wire x1="172.72" y1="121.92" x2="172.72" y2="124.46" width="0.1524" layer="91"/>
+<wire x1="172.72" y1="124.46" x2="180.34" y2="124.46" width="0.1524" layer="91"/>
+<pinref part="P+2" gate="1" pin="+5V"/>
+<wire x1="180.34" y1="124.46" x2="180.34" y2="127" width="0.1524" layer="91"/>
+<pinref part="R4" gate="A" pin="2"/>
+<wire x1="180.34" y1="121.92" x2="180.34" y2="124.46" width="0.1524" layer="91"/>
+<junction x="180.34" y="124.46"/>
+<pinref part="R3" gate="A" pin="2"/>
+<wire x1="187.96" y1="121.92" x2="187.96" y2="124.46" width="0.1524" layer="91"/>
+<wire x1="187.96" y1="124.46" x2="180.34" y2="124.46" width="0.1524" layer="91"/>
+</segment>
+<segment>
+<pinref part="P+3" gate="1" pin="+5V"/>
+<pinref part="C5" gate="A" pin="1"/>
+<wire x1="205.74" y1="127" x2="205.74" y2="116.84" width="0.1524" layer="91"/>
+<pinref part="J2" gate="A" pin="VCC"/>
+<wire x1="205.74" y1="116.84" x2="205.74" y2="114.3" width="0.1524" layer="91"/>
+<wire x1="231.14" y1="116.84" x2="205.74" y2="116.84" width="0.1524" layer="91"/>
+<junction x="205.74" y="116.84"/>
+</segment>
+<segment>
 <wire x1="60.96" y1="116.84" x2="116.84" y2="116.84" width="0.1524" layer="91"/>
 <wire x1="116.84" y1="116.84" x2="116.84" y2="119.38" width="0.1524" layer="91"/>
@@
 <pinref part="P+1" gate="1" pin="+5V"/>
 <wire x1="116.84" y1="127" x2="116.84" y2="121.92" width="0.1524" layer="91"/>
-</segment>
-<segment>
-<pinref part="R5" gate="A" pin="2"/>
-<wire x1="172.72" y1="121.92" x2="172.72" y2="124.46" width="0.1524" layer="91"/>
-<wire x1="172.72" y1="124.46" x2="180.34" y2="124.46" width="0.1524" layer="91"/>
-<pinref part="P+2" gate="1" pin="+5V"/>
-<wire x1="180.34" y1="124.46" x2="180.34" y2="127" width="0.1524" layer="91"/>
-<pinref part="R4" gate="A" pin="2"/>
-<wire x1="180.34" y1="121.92" x2="180.34" y2="124.46" width="0.1524" layer="91"/>
-<junction x="180.34" y="124.46"/>
-<pinref part="R3" gate="A" pin="2"/>
-<wire x1="187.96" y1="121.92" x2="187.96" y2="124.46" width="0.1524" layer="91"/>
-<wire x1="187.96" y1="124.46" x2="180.34" y2="124.46" width="0.1524" layer="91"/>
-</segment>
-<segment>
-<pinref part="P+3" gate="1" pin="+5V"/>
-<pinref part="C5" gate="A" pin="1"/>
-<wire x1="205.74" y1="127" x2="205.74" y2="116.84" width="0.1524" layer="91"/>
-<pinref part="J2" gate="A" pin="VCC"/>
-<wire x1="205.74" y1="116.84" x2="205.74" y2="114.3" width="0.1524" layer="91"/>
-<wire x1="231.14" y1="116.84" x2="205.74" y2="116.84" width="0.1524" layer="91"/>
-<junction x="205.74" y="116.84"/>
-</segment>
-</net>
+<pinref part="J1" gate="A" pin="VBUS"/>
+</segment>
+</net>
